File: Boards/ProgrammaGull_E3/ProgrammaGull_E3/ProgrammaGull_E3.kicad_pcb (KiCad board)
At the start: 2 copper layers, 45 parts, among them J1 Conn_01x12_Pin, J2 Conn_02x04_Counter_Clockwise, J3 Conn_01x12_Pin, J4 Conn_01x12_Pin, J5 Conn_01x12_Pin, U1 ICE40UP5K-SG48ITR, U2 W25Q32JVZP, U3 AP2127K-3.3, U4 AP2127K-2.5, U6 AP2127K-1.2

Commit message: Initial Sandpiper Commit
Parts:
- removed C1, C10, C11, C12, C13, C14, C15, C19, C21, C4, C9: 2u2, Capacitor_SMD:C_0603_1608Metric_Pad1.08x0.95mm_HandSolder
- removed C16, C17, C18, C2, C20, C22, C5, C7: 100n, Capacitor_SMD:C_0603_1608Metric_Pad1.08x0.95mm_HandSolder
- removed C3, C6, C8: 10n, Capacitor_SMD:C_0603_1608Metric_Pad1.08x0.95mm_HandSolder
- removed D1: 1N4148WT, Diode_SMD:D_SOD-523
- removed D3: LED_AGBR, LED_SMD:LED_Cree-PLCC4_2x2mm_CW
- removed J1, J3, J4, J5: Conn_01x12_Pin, Connector_PinSocket_2.54mm:PinSocket_1x12_P2.54mm_Vertical
- removed J2: Conn_02x04_Counter_Clockwise, Connector_PinSocket_2.54mm:PinSocket_2x04_P2.54mm_Vertical
- removed R1, R2, R3, R4, R5, R6, R8: R_Small, Resistor_SMD:R_0603_1608Metric_Pad0.98x0.95mm_HandSolder
- removed R10, R11, R9: 10k, Resistor_SMD:R_0603_1608Metric_Pad0.98x0.95mm_HandSolder
- removed R7: 100R, Resistor_SMD:R_0603_1608Metric_Pad0.98x0.95mm_HandSolder
- removed U1: ICE40UP5K-SG48ITR, Package_DFN_QFN:QFN-48-1EP_7x7mm_P0.5mm_EP5.6x5.6mm
- removed U2: W25Q32JVZP, Package_SON:WSON-8-1EP_6x5mm_P1.27mm_EP3.4x4.3mm
- removed U3: AP2127K-3.3, Package_TO_SOT_SMD:SOT-23-5
- removed U4: AP2127K-2.5, Package_TO_SOT_SMD:SOT-23-5
- removed U6: AP2127K-1.2, Package_TO_SOT_SMD:SOT-23-5
Routing:
- net /IOB_18a: track 21.9 -> 0.00 mm
- net /IOB_16a: track 21.0 -> 0.00 mm
- net /IOB_20a: track 20.2 -> 0.00 mm
- net /~{CRESET}: track 19.2 -> 0.00 mm
- net /IOB_22a: track 18.4 -> 0.00 mm
- net /CDONE: track 17.3 -> 0.00 mm
- net /IOB_13b: track 15.4 -> 0.00 mm
- net /IOB_8a: track 14.0 -> 0.00 mm
- net /IOB_9b: track 12.2 -> 0.00 mm
- net /IOB_4a: track 11.6 -> 0.00 mm
- net /IOB_2a: track 11.1 -> 0.00 mm
- net /IOB_6a: track 10.5 -> 0.00 mm
- net /IOB_0a: track 10.2 -> 0.00 mm
- net /IOT_49a: track 9.43 -> 0.00 mm
- net /IOB_5b: track 9.39 -> 0.00 mm
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Other:
- copper layers 2 -> 4
