File: Boards/ProgrammaGull_E3/ProgrammaGull_E3/ProgrammaGull_E3.kicad_sch (KiCad schematic)
At the start: 45 parts, among them J1 Conn_01x12_Pin, J2 Conn_02x04_Counter_Clockwise, J3 Conn_01x12_Pin, J4 Conn_01x12_Pin, J5 Conn_01x12_Pin, U1 ICE40UP5K-SG48ITR, U2 W25Q32JVZP, U3 AP2127K-3.3, U4 AP2127K-2.5, U6 AP2127K-1.2

Commit message: Initial Sandpiper Commit
Parts:
- removed J1, J3, J4, J5: Conn_01x12_Pin, Connector_PinSocket_2.54mm:PinSocket_1x12_P2.54mm_Vertical, symbol Connector:Conn_01x12_Pin
- removed R4, R5, R8: R_Small, Resistor_SMD:R_0603_1608Metric_Pad0.98x0.95mm_HandSolder, symbol Device:R_Small
- removed U2: W25Q32JVZP, Package_SON:WSON-8-1EP_6x5mm_P1.27mm_EP3.4x4.3mm, symbol Memory_Flash:W25Q32JVZP
- added C23, C25, C27, C28, C29, C35, C36: 1u, Capacitor_SMD:C_0603_1608Metric_Pad1.08x0.95mm_HandSolder, symbol Device:C_Small
- added C24, C30, C31, C32: 100n, Capacitor_SMD:C_0603_1608Metric_Pad1.08x0.95mm_HandSolder, symbol Device:C_Small
- added C26, C33, C34: 2u2, Capacitor_SMD:C_0603_1608Metric_Pad1.08x0.95mm_HandSolder, symbol Device:C_Small
- added J1, J3: Conn_01x24_Pin, Connector_PinSocket_2.54mm:PinSocket_1x24_P2.54mm_Vertical, symbol Connector:Conn_01x24_Pin
- added R12, R8: 100R, Resistor_SMD:R_0603_1608Metric_Pad0.98x0.95mm_HandSolder, symbol Device:R_Small_US
- added R4, R5: 10k, Resistor_SMD:R_0603_1608Metric_Pad0.98x0.95mm_HandSolder, symbol Device:R_Small_US
- added RN1, RN2: 10k, Resistor_SMD:R_Array_Convex_2x0603, symbol Device:R_Pack02
- added U2: W25Q32JVSS, Package_SO:SOIC-8_5.23x5.23mm_P1.27mm, symbol Memory_Flash:W25Q32JVSS
- added U5: ~, ProgrammaGull_Logic:TDFN-16-1EP_3x2_mm, symbol ProgrammaGull_Logic:MAX11192ATE+T
- added U7: LM324A, Package_SO:TSSOP-14_4.4x5mm_P0.65mm, symbol Amplifier_Operational:LM324A
- added U8: ~, Package_CSP:LFCSP-WD-10-1EP_3x3mm_P0.5mm_EP1.64x2.38mm, symbol ProgrammaGull_Logic:AD9837
Connections:
- net +3V3: now also C21.1, D3.1 (A), C23.1, C24.1, C25.1, C26.1, C32.1, J3.1 (Pin_1), J3.2 (Pin_2), U5.15 (AVDD), U5.9 (OVDD), U7.4 (V+)
- net +5V: now also J1.1 (Pin_1)
- net BANK_0_V+: now also J3.13 (Pin_13)
- net BANK_1_V+: now also J1.3 (Pin_3), U2.8 (VCC)
- net BANK_2_V+: now also J1.4 (Pin_4)
- net CDONE: now also J1.10 (Pin_10)
- net FLASH_IO2: now also U2.3 (IO2)
- net FLASH_IO3: now also U2.7 (IO3)
- net GND: now also C23.2, C24.2, C25.2, C26.2, C27.2, C28.2, C29.2, C30.2, C31.2, C32.2, C33.2, C34.2, J1.2 (Pin_2), J3.10 (Pin_10), J3.3 (Pin_3), J3.4 (Pin_4), RN1.4 (R1.2), RN2.4 (R1.2), U2.4 (GND), U5.12 (REFGND), U5.16 (AGND), U5.17 (EP), U5.6 (OGND), U7.11 (V-)
- net IOB_0a: now also J3.23 (Pin_23), U5.7 (DOUT1)
- net IOB_13b: now also J1.9 (Pin_9)
- net IOB_16a: now also J1.12 (Pin_12)
- net IOB_18a: now also J1.13 (Pin_13)
- net IOB_20a: now also J1.14 (Pin_14)
- net IOB_22a: now also J1.15 (Pin_15)
- net IOB_23b: now also J1.20 (Pin_20)
- net IOB_24a: now also J1.16 (Pin_16)
- net IOB_25b_G3: now also J1.19 (Pin_19)
- net IOB_29b: now also J1.18 (Pin_18)
- net IOB_2a: now also J3.24 (Pin_24), U5.8 (DOUT2)
- net IOB_31b: now also J1.17 (Pin_17)
- net IOB_32a_SPI_SO: now also J1.21 (Pin_21), U2.2 (DO(IO1))
- net IOB_33b_SPI_SI: now also J1.24 (Pin_24), U2.5 (DI(IO0))
- net IOB_34a_SPI_SCK: now also J1.22 (Pin_22), U2.6 (CLK)
- net IOB_35b_SPI_SS: now also J1.23 (Pin_23), U2.1 (~{CS})
- net IOB_3b_G6: now also J3.21 (Pin_21)
- net IOB_4a: now also J1.5 (Pin_5), U5.10 (SCK)
- net IOB_5b: now also J3.22 (Pin_22), U5.5 (~{CVTST})
- net IOB_6a: now also J1.6 (Pin_6)
- net IOB_8a: now also J1.8 (Pin_8)
- net IOB_9b: now also J1.7 (Pin_7)
- net IOT_36b: now also J3.6 (Pin_6)
- net IOT_37a: now also J3.5 (Pin_5)
- net IOT_38b: now also J3.8 (Pin_8)
- net IOT_39a: now also J3.7 (Pin_7)
- net IOT_41a: now also J3.9 (Pin_9)
- net IOT_42b: now also J3.11 (Pin_11)
- net IOT_43a: now also J3.12 (Pin_12)
- net IOT_44b: now also J3.14 (Pin_14)
- net IOT_45a_G1: now also J3.17 (Pin_17)
- net IOT_46b_G0: now also J3.15 (Pin_15)
- net IOT_48b: now also J3.16 (Pin_16)
- net IOT_49a: now also J3.20 (Pin_20)
- net IOT_50b: now also J3.18 (Pin_18)
- net IOT_51a: now also J3.19 (Pin_19)
- net ~{CRESET}: now also J1.11 (Pin_11)
- new net: C27.1, U5.14 (REFIN/OUT)
- new net: C36.2, R5.2, U7.10 (+)
- new net: R12.1, U7.8, U7.9 (-)
- new net: R12.2, U5.3 (AIN2+)
- new net: RN1.1 (R1.1), RN1.2 (R2.1), U7.3 (+)
- new net: C35.2, R4.2, U7.12 (+)
- new net: RN2.1 (R1.1), RN2.2 (R2.1), U7.5 (+)
- new net: R8.2, U5.1 (AIN1+)
- new net: R8.1, U7.13 (-), U7.14
- new net ANALOG_IN_0: C35.1
- new net ANALOG_IN_1: C36.1
- new net REF1_ADC: C28.1, RN1.3 (R2.2), U5.13 (REF1)
- new net REF1/2_BIAS: C30.1, C33.1, R4.1, U5.2 (AIN1-), U7.1, U7.2 (-)
- new net REF2_ADC: C29.1, RN2.3 (R2.2), U5.11 (REF2)
- new net REF2/2_BIAS: C31.1, C34.1, R5.1, U5.4 (AIN2-), U7.6 (-), U7.7
Other:
- note added: "Dual Simultaneous Sampling 12/14/16 bit ADC MAX11192-MAX11198 Inputs AC coupled and biased to VREF/2 Differential 2's complement input"
- note added: "Input Bias Offsets and external bias voltage feed"
- note added: "Matched pair or array"
- note added: "Rin = 10k f_hp = 1 / (2pi R * C) f_hp = 1 / (2pi * 10k * 1u) f_hp = 15.91 Hz"
