File: Boards/ProgrammaGull_Sandpiper/ProgrammaGull_Sandpiper/ProgrammaGull_Sandpiper.kicad_pcb (KiCad board)
At the start: 4 copper layers, 100 x 75 mm, 183 parts, among them J4 Conn_01x22_Socket, P1 USB_C_Plug_USB2.0, Q1 MMBT2907, Q2 MMBT2907, Q3 MMBT2907, Q4 MMBT2907, Q5 MMBT2907, Q6 MMBT2907, Q7 MMBT2907, Q8 MMBT2907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

Commit message: Fixed 7 segment drive circuitry to work properly, swap to 74 596 + segment brightness limiting resistors
Parts:
- removed U9: 74AHC595, Package_SO:TSSOP-16_4.4x5mm_P0.65mm
- added C3: 1u, Capacitor_SMD:C_0603_1608Metric, F.Cu at (65.3, 75.1)
- added R2: 680R, Resistor_SMD:R_0603_1608Metric, F.Cu at (71.0, 48.9)
- added R35: 680R, Resistor_SMD:R_0603_1608Metric, F.Cu at (50.2, 50.2)
- added R87: 680R, Resistor_SMD:R_0603_1608Metric, F.Cu at (53.3, 49.0)
- added R88: 680R, Resistor_SMD:R_0603_1608Metric, F.Cu at (75.0, 50.4)
- added R89: 680R, Resistor_SMD:R_0603_1608Metric, F.Cu at (61.0, 47.3)
- added R90: 680R, Resistor_SMD:R_0603_1608Metric, F.Cu at (75.0, 52.0)
- added R91: 680R, Resistor_SMD:R_0603_1608Metric, F.Cu at (66.2, 47.3)
- added U3: 74HC596, Package_SO:TSSOP-16_4.4x5mm_P0.65mm, F.Cu at (66.8, 54.0)
- R54: value 10k -> 680R
- moved R54 12.6 mm to (75.0, 48.9), turned to 180 degrees
- moved Q3 1.50 mm to (63.5, 44.5)
- moved R70 1.50 mm to (63.6, 47.3)
- moved C2 0.38 mm to (58.9, 71.6)
- moved D1 0.38 mm to (62.8, 71.1)
- moved U5 0.38 mm to (62.5, 74.0)
Connections:
- R54 pad 1: GND -> /UI_LSB_CA1
Routing:
- net +1V2: track 20.6 -> 37.4 mm, vias 0 -> 2
- net /UI_MSB_CA0: track 23.3 -> 6.78 mm
- net Net-(U3-QH): track 0.00 -> 15.4 mm
- net Net-(U3-QG): track 0.00 -> 13.1 mm
- net /UI_MSB_CA1: track 20.4 -> 8.11 mm
- net /UI_LSB_CA3: track 45.3 -> 33.5 mm
- net /~{UI_7SEGSR_OE}: track 27.9 -> 36.5 mm, vias 2 -> 3
- net Net-(U3-QA): track 0.00 -> 8.38 mm
- net /UI_LSB_CA1: track 11.7 -> 3.54 mm
- net GND: track 111.3 -> 119.4 mm, vias 95 -> 96
- net Net-(U3-QF): track 0.00 -> 7.42 mm
- net /UI_LSB_CA2: track 33.6 -> 27.1 mm
- net Net-(U3-QB): track 0.00 -> 5.41 mm
- net /UI_LSB_CA0: track 8.75 -> 3.56 mm
- net Net-(U3-QD): track 0.00 -> 4.53 mm
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Other:
- outline, holes or cut-outs redrawn
- board text added: "ProgrammaGull Logic Sandpiper Joseph A. De Vico 11/06/2023"
- board text added: "Version: Alpha 0.1"
- board text added: "iCE40-UP5k SG-48"
