File: Boards/ProgrammaGull_Sandpiper/ProgrammaGull_Sandpiper/ProgrammaGull_Sandpiper.kicad_sch (KiCad schematic)
At the start: 13 parts, among them P1 USB_C_Plug_USB2.0, U1 ICE40UP5K-SG48ITR, U2 W25Q32JVZP, U3 MIC5504-3.3YM5, U4 MIC5504-1.2YM5, U5 MIC5504-2.5YM5, U6 FT232H

Commit message: Big Sandpiper updates :)
Parts:
- removed U6: FT232H, symbol Interface_USB:FT232H
- added C10, C12, C15, C17, C25, C27, C30: 4u7, symbol Device:C_Small
- added C11, C13, C14, C16, C18, C20, C22, C26, C28, C29, C8, C9: 100n, symbol Device:C_Small
- added C19, C21, C23, C24: 1u, symbol Device:C_Small
- added C7: 10u, symbol Device:C_Small
- added D1: 1N4148W, Diode_SMD:D_SOD-123, symbol Diode:1N4148W
- added D10: LED_ABGR, symbol Device:LED_ABGR
- added D2, D3, D4, D5, D6, D7, D8, D9: LED, symbol Device:LED
- added FB1, FB2: FerriteBead_Small, symbol Device:FerriteBead_Small
- added Q1, Q2, Q3, Q4: MMBT2222A, Package_TO_SOT_SMD:SOT-23, symbol Transistor_BJT:MMBT5550L
- added R1, R2: 27R, symbol Device:R_Small_US
- added R10, R12, R14, R16, R18, R20, R22, R24, R26, R28, R30, R32, R34, R35, R36, R37, R39, R40, R41, R42, R63, R65, R66, R67, R68, R69, R7, R70, R8: 10k, symbol Device:R_Small_US
- added R11, R13, R15, R17, R19, R21, R23, R25, R27, R29, R31, R55, R56, R57, R58, R59, R6, R60, R61, R62, R64, R9: 220R, symbol Device:R_Small_US
- added R3, R4: 56k, symbol Device:R_Small_US
- added R33: 2k2, symbol Device:R_Small_US
- added R38: 12k 1%, symbol Device:R_Small_US
- added R43, R44, R45, R46: 4k3, symbol Device:R_Small_US
- added R47, R48, R49, R5, R50, R51, R52, R53, R54: 100R, symbol Device:R_Small_US
- added SW1, SW2, SW3, SW4, SW5, SW6, SW7, SW8: SW_SPDT, symbol Switch:SW_SPDT
- added SW10, SW11, SW12, SW13, SW14, SW9: SW_Push, symbol Switch:SW_Push
- added U10: 74HCS596, symbol 74xx:74HCT596
- added U6: 93LCxxAxxOT, Package_TO_SOT_SMD:SOT-23-6, symbol Memory_EEPROM:93LCxxAxxOT
- added U7: FT2232HQ, Package_DFN_QFN:QFN-64-1EP_9x9mm_P0.5mm_EP4.35x4.35mm, symbol Interface_USB:FT2232HQ
- added U8: CC56-12YWA, Display_7Segment:CC56-12YWA, symbol Display_Character:CC56-12YWA
Connections:
- net +1V2: now also U1.30 (VCC), U1.5 (VCC), R5.2
- net +2V5: now also U1.24 (VPP_2V5), D1.1 (K)
- net +3V3: now also U1.1 (VCCIO_2), U1.22 (SPI_VCCIO1), U1.33 (VCCIO_0), U2.8 (VCC), C16.1, C17.1, C18.1, C19.1, C20.1, C21.1, C22.1, C23.1, C27.1, C28.1, C29.1, C30.1, C9.1, D1.2 (A), D10.1 (A), FB1.2, FB2.2, R10.2, R12.2, R14.2, R16.2, R18.2, R20.2, R32.2, R34.2, R35.2, R36.2, R37.2, R39.2, R40.2, R41.2, R42.2, R55.2, R56.2, R57.2, R58.2, R59.2, R60.2, R61.2, R62.2, R65.2, R7.2, R8.2, SW1.3 (C), SW10.1, SW11.1, SW12.1, SW13.1, SW14.1, SW2.3 (C), SW3.3 (C), SW4.3 (C), SW5.3 (C), SW6.3 (C), SW7.3 (C), SW8.3 (C), SW9.1, U10.16 (VCC), U6.6 (VCC), U7.20 (VCCIO), U7.31 (VCCIO), U7.42 (VCCIO), U7.50 (VREGIN), U7.56 (VCCIO)
- net GND: now also U1.49 (GND), U2.4 (GND), U2.9 (EP), C10.2, C11.2, C12.2, C13.2, C14.2, C15.2, C16.2, C17.2, C18.2, C19.2, C20.2, C21.2, C22.2, C23.2, C24.2, C25.2, C26.2, C27.2, C28.2, C29.2, C30.2, C7.2, C8.2, C9.2, Q1.2 (E), Q2.2 (E), Q3.2 (E), Q4.2 (E), R22.1, R24.1, R26.1, R28.1, R3.1, R30.1, R38.1, R4.1, R63.1, R66.1, R67.1, R68.1, R69.1, R70.1, SW1.1 (A), SW2.1 (A), SW3.1 (A), SW4.1 (A), SW5.1 (A), SW6.1 (A), SW7.1 (A), SW8.1 (A), U10.8 (GND), U6.2 (GND), U7.1 (GND), U7.10 (AGND), U7.11 (GND), U7.13 (TEST), U7.15 (GND), U7.25 (GND), U7.35 (GND), U7.47 (GND), U7.5 (GND), U7.51 (GND), U7.65 (GND)
- net VBUS: now also C24.1, C25.1, C26.1
- net FLASH_MOSI: now reaches U1.14 (IOB_32a_SPI_SO)
- net FLASH_MOSI: now also U2.5 (DI(IO0)), U7.17 (ADBUS1)
- net FLASH_SCK: now reaches U1.15 (IOB_34a_SPI_SCK)
- net FLASH_SCK: now also U2.6 (CLK), R42.1, U7.16 (ADBUS0)
- net FLASH_CS: now reaches U1.16 (IOB_35b_SPI_SS)
- net FLASH_CS: now also U2.1 (~{CS}), R32.1, U7.21 (ADBUS4)
- net FLASH_MISO: now reaches U1.17 (IOB_33b_SPI_SI)
- net FLASH_MISO: now also U2.2 (DO(IO1)), U7.18 (ADBUS2)
- net ~{UI_ULEDSR_CLR}: now reaches U1.19 (IOB_29b)
- net ~{UI_ULEDSR_CLR}: now also R65.1, U10.10 (~{SRCLR})
- net UI_ULEDSR_CLK: now reaches U1.20 (IOB_25b_G3)
- net UI_ULEDSR_CLK: now also U10.11 (SRCLK)
- net UI_ULEDSR_DIN: now reaches U1.21 (IOB_23b)
- net UI_ULEDSR_DIN: now also U10.14 (SER)
- net UP5K_CDONE: now reaches U1.7 (CDONE)
- net UP5K_CDONE: now also U7.23 (ADBUS6)
- net UP5K_CRESET: now reaches U1.8 (~{CRESET})
- net UP5K_CRESET: now also U7.24 (ADBUS7)
- net at U1.29 (VCCPLL): now also C7.1, C8.1, R5.1
- net at U2.3 (IO2): now also R40.1
- net at U2.7 (IO3): now also R41.1
- net USB_CC: now reaches P1.A5 (CC)
- net USB_CC: now also R3.2
- net at P1.A6 (D+): now also R2.1
- net at P1.A7 (D-): now also R1.1
- net USB_VCONN: now reaches P1.B5 (VCONN)
- net USB_VCONN: now also R4.2
- net UI_AUX_BUTTON: now reaches U1.23 (IOT_37a)
- net UI_AUX_BUTTON: now also R64.1
- net UI_SW7: now reaches U1.25 (IOT_36b)
- net UI_SW7: now also R6.2
- net UI_SW6: now reaches U1.26 (IOT_39a)
- net UI_SW6: now also R9.2
- net UI_SW5: now reaches U1.27 (IOT_38b)
- net UI_SW5: now also R11.2
- net UI_SW4: now reaches U1.28 (IOT_41a)
- net UI_SW4: now also R13.2
- net UI_SW3: now reaches U1.31 (IOT_42b)
- net UI_SW3: now also R15.2
- net UI_SW2: now reaches U1.32 (IOT_43a)
- net UI_SW2: now also R17.2
- net UI_SW1: now reaches U1.34 (IOT_44b)
- net UI_SW1: now also R19.2
- net UI_SW0: now reaches U1.35 (IOT_46b_G0)
- net UI_SW0: now also R21.2
- net UI_DPAD_C: now reaches U1.36 (IOT_48b)
- net UI_DPAD_C: now also R31.1
- net UI_DPAD_L: now reaches U1.37 (IOT_45a_G1)
- net UI_DPAD_L: now also R29.1
- net UI_DPAD_U: now reaches U1.38 (IOT_50b)
- net UI_DPAD_U: now also R23.1
- net UI_RGBLED_G: now reaches U1.39 (RGB0)
- net UI_RGBLED_G: now also D10.3 (GK)
- net UI_RGBLED_B: now reaches U1.40 (RGB1)
- net UI_RGBLED_B: now also D10.2 (BK)
- net UI_RGBLED_R: now reaches U1.41 (RGB2)
- net UI_RGBLED_R: now also D10.4 (RK)
- net UI_DPAD_D: now reaches U1.42 (IOT_51a)
- net UI_DPAD_D: now also R25.1
- net UI_DPAD_R: now reaches U1.43 (IOT_49a)
- net UI_DPAD_R: now also R27.1
- new net: R10.1, R11.1, SW3.2 (B)
- new net: R20.1, R21.1, SW8.2 (B)
- new net: D4.2 (A), R57.1
- new net: D7.2 (A), R60.1
- new net: R14.1, R15.1, SW5.2 (B)
- new net: Q1.1 (B), R43.1
- new net: Q1.3 (C), U8.6 (CC4)
- new net: R26.2, R27.2, SW11.2
- new net: R28.2, R29.2, SW12.2
- new net: R38.2, U7.6 (REF)
- new net: R18.1, R19.1, SW7.2 (B)
- new net: D8.2 (A), R61.1
- new net: C12.1, C13.1, FB1.1, U7.9 (VPLL)
- new net: Q3.1 (B), R45.1
- new net: Q3.3 (C), U8.9 (CC2)
- new net: D9.2 (A), R62.1
- new net: R6.1, R7.1, SW1.2 (B)
- new net: R39.1, U7.14 (~{RESET})
- new net: C14.1, C15.1, FB2.1, U7.4 (VPHY)
- new net: R24.2, R25.2, SW10.2
- new net: D5.2 (A), R58.1
- new net: R50.1, U8.4 (c)
- new net: D3.2 (A), R56.1
- new net: R16.1, R17.1, SW6.2 (B)
- new net: R54.2, U8.3 (DPX)
- new net: R30.2, R31.2, SW13.2
- new net: D2.2 (A), R55.1
- new net: D6.2 (A), R59.1
- new net: R47.1, U8.11 (a)
- new net: R51.2, U8.1 (e)
- new net: R52.2, U8.10 (f)
- new net: Q4.3 (C), U8.12 (CC1)
- new net: R49.1, U8.2 (d)
- new net: R53.2, U8.5 (g)
- new net: R48.1, U8.7 (b)
- new net: Q2.3 (C), U8.8 (CC3)
- new net: R12.1, R13.1, SW4.2 (B)
- new net: R63.2, R64.2, SW14.2
- new net: R8.1, R9.1, SW2.2 (B)
- new net: Q2.1 (B), R44.1
- new net: Q4.1 (B), R46.1
- new net: R22.2, R23.2, SW9.2
- new net +1V8: C10.1, C11.1, U7.12 (VCORE), U7.37 (VCORE), U7.49 (VREGOUT), U7.64 (VCORE)
- new net CLK_12M: U7.2 (OSCI)
- new net EEPROM_SPI_CLK: R36.1, U6.4 (CLK), U7.62 (EECLK)
- new net EEPROM_SPI_CS: R34.1, R35.1, U6.5 (CS), U7.63 (EECS)
- new net EEPROM_SPI_DI: R33.2, U6.3 (DI), U7.61 (EEDATA)
- new net EEPROM_SPI_DO: R33.1, R37.1, U6.1 (DO)
- new net UI_LED_0: D9.1 (K), U10.15 (QA)
- new net UI_LED_1: D8.1 (K), U10.1 (QB)
- new net UI_LED_2: D7.1 (K), U10.2 (QC)
- new net UI_LED_3: D6.1 (K), U10.3 (QD)
- new net UI_LED_4: D5.1 (K), U10.4 (QE)
- new net UI_LED_5: D4.1 (K), U10.5 (QF)
- new net UI_LED_6: D3.1 (K), U10.6 (QG)
- new net UI_LED_7: D2.1 (K), U10.7 (QH)
- new net UI_SEG0_CC: R46.2, R70.2
- new net UI_SEG1_CC: R45.2, R69.2
- new net UI_SEG2_CC: R44.2, R67.2
- new net UI_SEG3_CC: R43.2, R68.2
- new net UI_SEG_A: R47.2
- new net UI_SEG_B: R48.2
- new net UI_SEG_C: R50.2
- new net UI_SEG_D: R49.2
- new net UI_SEG_DP: R54.1
- new net UI_SEG_E: R51.1
- new net UI_SEG_F: R52.1
- new net UI_SEG_G: R53.1
- new net UP5K_UART_CTS: U7.41 (BDBUS3)
- new net UP5K_UART_DCD: U7.45 (BDBUS6)
- new net UP5K_UART_DSR: U7.44 (BDBUS5)
- new net UP5K_UART_DTR: U7.43 (BDBUS4)
- new net UP5K_UART_RTS: U7.40 (BDBUS2)
- new net UP5K_UART_RX: U7.38 (BDBUS0)
- new net UP5K_UART_TX: U7.39 (BDBUS1)
- new net USB_D+: R2.2, U7.8 (DP)
- new net USB_D-: R1.2, U7.7 (DM)
- new net ~{UI_ULEDSR_OE}: R66.2, U10.13 (~{OE})
- no-connect marks 0 -> 24
Other:
- note added: "4 Char 7 Segment Display"
- note added: "As rated can drive each LED at ~8mA"
- note added: "BJT: 7seg * 15mA ~= 100mA 2222A @ 100mA, Vbe = 3.3 -> Rb ~= 4500 ~= 1% tol 4k3"
- note added: "D Pad"
- note added: "Default State: Output Enabled, Clear Disabled"
- note added: "FPGA Core Power"
- note added: "FPGA Pinout"
- note added: "LC Filter action as recommended in datasheet"
- note added: "NOTE: RX and TX are from the iCE40-UP5k Perspective!!"
- note added: "Open-Drain 74 Logic Use HCS Leave push/pull floating"
- note added: "Rec Part: LCSC SR420361N"
- note added: "SPI Flash"
- note added: "SWAP TO CA AND USE OPEN COLLECTOR SHIFT REG!!!!"
- note added: "Segment: Vf = 2.0V If = 15mA Rser = (3.3V - 2.0V) / 0.015A = 86.66 ~= 100 ohm"
- note added: "Serial UI Bank - User LED and 7 Segment"
- note added: "Slanted to annoy Alec :)"
- note added: "Switch Bank"
- note added: "UI Bank - Switches, Buttons, RGB LED"
- note added: "USB Prog and VCOM"
- note added: "User LED Bank, Serial Access"
- note added: "https://datasheet.lcsc.com/lcsc/1810281611_ARKLED-Wuxi-ARK-Tech-Elec-SR420361N_C98926.pdf"
- moved on the sheet: C2, C3, C5, C6, U1A, U1B, U1C, U1D, U2, U4, U5

Commit message: Sandpiper Progress!
Parts:
- removed Q1, Q2, Q3, Q4: MMBT2222A, Package_TO_SOT_SMD:SOT-23, symbol Transistor_BJT:MMBT5550L
- removed U10: 74HCS596, symbol 74xx:74HCT596
- removed U8: CC56-12YWA, Display_7Segment:CC56-12YWA, symbol Display_Character:CC56-12YWA
- added C31, C32, C34, C36, C37, C38, C39: 100n, symbol Device:C_Small
- added C33, C35: 4u7, symbol Device:C_Small
- added Q1, Q2, Q3, Q4, Q5, Q6, Q7, Q8: MMBT2907, Package_TO_SOT_SMD:SOT-23, symbol Transistor_BJT:MMBT3906
- added R71, R72, R73, R74, R75, R78: 10k, symbol Device:R_Small_US
- added R76, R77: 2k2, symbol Device:R_Small_US
- added SW15: RotaryEncoder, symbol Device:RotaryEncoder
- added U10, U8: ~, symbol ProgrammaGull_Logic:MHDA3641SRBW
- added U12: 74HC596, symbol 74xx:74HC596
- added U13, U9: 74AHC595, symbol 74xx:74AHC595
- R43, R44, R45, R46: value 4k3 -> 383R
- R47, R48, R49, R50: value 100R -> 383R
- R51, R52, R53, R54: value 100R -> 10k
Connections:
- net +3V3: now also R51.2, R52.2, R53.2, C32.1, C33.1, C34.1, C35.1, R75.2, R78.2, U12.16 (VCC), U13.16 (VCC), U9.16 (VCC); no longer R55.2, R56.2, R57.2, R58.2, R59.2, R60.2, R61.2, R62.2
- net GND: now also D2.1 (K), D3.1 (K), D4.1 (K), D5.1 (K), D6.1 (K), D7.1 (K), D8.1 (K), D9.1 (K), R54.1, C31.2, C32.2, C33.2, C34.2, C35.2, C36.2, C37.2, C38.2, C39.2, SW15.C, U12.8 (GND), U13.8 (GND), U9.8 (GND); no longer R67.1, R68.1, R69.1, R70.1
- net UI_LED_0: now also R62.2, U13.15 (QA); no longer D9.1 (K)
- net UI_LED_1: now also R61.2, U13.1 (QB); no longer D8.1 (K)
- net UI_LED_2: now also R60.2, U13.2 (QC); no longer D7.1 (K)
- net UI_LED_3: now also R59.2, U13.3 (QD); no longer D6.1 (K)
- net UI_LED_4: now also R58.2, U13.4 (QE); no longer D5.1 (K)
- net UI_LED_5: now also R57.2, U13.5 (QF); no longer D4.1 (K)
- net UI_LED_6: now also R56.2, U13.6 (QG); no longer D3.1 (K)
- net UI_LED_7: now also R55.2, U13.7 (QH); no longer D2.1 (K)
- net UI_SEG_A: now also R43.1, U10.11 (A), U8.11 (A); no longer R47.2
- net UI_SEG_B: now also R44.1, U10.7 (B), U8.7 (B); no longer R48.2
- net UI_SEG_C: now also R45.1, U10.4 (C), U8.4 (C); no longer R50.2
- net UI_SEG_D: now also R46.1, U10.2 (D), U8.2 (D); no longer R49.2
- net UI_SEG_DP: now also R50.1, U10.3 (DP), U8.3 (DP); no longer R54.1
- net UI_SEG_E: now also R47.1, U10.1 (E), U8.1 (E); no longer R51.1
- net UI_SEG_F: now also R48.1, U10.10 (F), U8.10 (F); no longer R52.1
- net UI_SEG_G: now also R49.1, U10.5 (G), U8.5 (G); no longer R53.1
- net UI_ULEDSR_CLK: now also U13.11 (SRCLK), U13.12 (RCLK)
- net UI_ULEDSR_DIN: now also U13.14 (SER)
- net VBUS: now also R67.2, R68.2, R69.2, R70.2, Q1.2 (E), Q2.2 (E), Q3.2 (E), Q4.2 (E), Q5.2 (E), Q6.2 (E), Q7.2 (E), Q8.2 (E), R71.2, R72.2, R73.2, R74.2
- net ~{UI_ULEDSR_CLR}: now also C31.1, U13.10 (~{SRCLR}); no longer U1.19 (IOB_29b)
- net ~{UI_ULEDSR_OE}: now also U13.13 (~{OE})
- net UI_7SEGSR_DIN: now reaches U1.10 (IOB_18a)
- net UI_7SEGSR_DIN: now also U12.14 (SER)
- net UI_7SEGSR_CLK: now reaches U1.11 (IOB_20a)
- net UI_7SEGSR_CLK: now also U12.11 (SRCLK), U9.11 (SRCLK)
- net UI_7SEGSR_RCLK: now reaches U1.12 (IOB_22a)
- net UI_7SEGSR_RCLK: now also U12.12 (RCLK), U9.12 (RCLK)
- net ~{UI_7SEGSR_OE}: now reaches U1.13 (IOB_24a)
- net ~{UI_7SEGSR_OE}: now also R53.1, U9.13 (~{OE})
- net UI_ROTENC_B: now reaches U1.18 (IOB_31b)
- net UI_ROTENC_B: now also R77.2
- net at R54.2: now also U12.13 (~{OE})
- net UI_SEG0_CC: no longer names the net of R46.2
- net UI_SEG0_CC: now also U12.3 (QD); no longer R70.2
- net UI_SEG1_CC: no longer names the net of R45.2
- net UI_SEG1_CC: now also U12.2 (QC); no longer R69.2
- net UI_SEG2_CC: no longer names the net of R44.2
- net UI_SEG2_CC: now also U12.1 (QB); no longer R67.2
- net UI_SEG3_CC: no longer names the net of R43.2
- net UI_SEG3_CC: now also U12.15 (QA); no longer R68.2
- new net: C39.1, R77.1, R78.1, SW15.B
- new net: Q5.3 (C), U10.12 (CA0)
- new net: Q6.3 (C), U10.9 (CA1)
- new net: C37.1, R52.1, U12.10 (~{SRCLR})
- new net: R47.2, U12.4 (QE)
- new net: R48.2, U12.5 (QF)
- new net: R49.2, U12.6 (QG)
- new net: R50.2, U12.7 (QH)
- new net: C38.1, R75.1, R76.1, SW15.A
- new net: Q2.3 (C), U8.9 (CA1)
- new net: Q3.3 (C), U8.8 (CA2)
- new net: C36.1, R51.1, U9.10 (~{SRCLR})
- new net: Q1.3 (C), U8.12 (CA0)
- new net: Q4.3 (C), U8.6 (CA3)
- new net: Q8.3 (C), U10.6 (CA3)
- new net: Q7.3 (C), U10.8 (CA2)
- new net UI_7SEG_SER_CARRY: U12.9 (QH'), U9.14 (SER)
- new net UI_LSB_CA0: Q5.1 (B), R71.1, U9.15 (QA)
- new net UI_LSB_CA1: Q6.1 (B), R72.1, U9.1 (QB)
- new net UI_LSB_CA2: Q7.1 (B), R73.1, U9.2 (QC)
- new net UI_LSB_CA3: Q8.1 (B), R74.1, U9.3 (QD)
- new net UI_MSB_CA0: Q1.1 (B), R67.1, U9.4 (QE)
- new net UI_MSB_CA1: Q2.1 (B), R68.1, U9.5 (QF)
- new net UI_MSB_CA2: Q3.1 (B), R70.1, U9.6 (QG)
- new net UI_MSB_CA3: Q4.1 (B), R69.1, U9.7 (QH)
- new net UI_ROTENC_A: R76.2, U1.19 (IOB_29b)
Other:
- note added: "8 Digit Common Anode 7 Segment Display!"
- note added: "Aux. User Button"
- note added: "Default State: Output Enabled Clear Disabled (after startup clr)"
- note added: "Keep OE disabled such that CA transistors are disabled by default."
- note added: "Note: THIS IS OPEN DRAIN"
- note added: "Note: THIS IS PUSH PULL"
- note added: "RGB LED"
- note added: "Rec Part: LCSC MHDA3641SRBW"
- note added: "Rotary Encoder"
- note added: "Serial UI Bank: User LED Bank 7 Segment Display"
- note added: "Shift with SRCLK, Add extra clk to update outputs properly. See: Sect. 8.1 in Datasheet RCLK tied to SRCLK"
- note added: "UI Bank: Switches Buttons RGB LED"
- note added: "https://datasheet.lcsc.com/lcsc/1912111437_MEIHUA-MHDA3641SRBW_C401125.pdf"
- note added: "https://www.ti.com/lit/ds/symlink/sn74hcs595.pdf"
- note added: "https://www.ti.com/lit/ds/symlink/sn74hcs596.pdf"
- note removed: "4 Char 7 Segment Display"
- note removed: "BJT: 7seg * 15mA ~= 100mA 2222A @ 100mA, Vbe = 3.3 -> Rb ~= 4500 ~= 1% tol 4k3"
- note removed: "Default State: Output Enabled, Clear Disabled"
- note removed: "Open-Drain 74 Logic Use HCS Leave push/pull floating"
- note removed: "Rec Part: LCSC SR420361N"
- note removed: "SWAP TO CA AND USE OPEN COLLECTOR SHIFT REG!!!!"
- note removed: "Segment: Vf = 2.0V If = 15mA Rser = (3.3V - 2.0V) / 0.015A = 86.66 ~= 100 ohm"
- note removed: "Serial UI Bank - User LED and 7 Segment"
- note removed: "UI Bank - Switches, Buttons, RGB LED"
- note removed: "https://datasheet.lcsc.com/lcsc/1810281611_ARKLED-Wuxi-ARK-Tech-Elec-SR420361N_C98926.pdf"
- moved on the sheet: C27, C28, C29, C30, D10, D2, D3, D4, D5, D6, D7, D8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

Commit message: Alpha Sandpiper Board Completegit status
Parts:
- removed R2: 27R, symbol Device:R_Small_US
- removed R35: 10k, symbol Device:R_Small_US
- removed SW1, SW2, SW3, SW4, SW5, SW6, SW7, SW8: SW_SPDT, symbol Switch:SW_SPDT
- removed U2: W25Q32JVZP, Package_SON:WSON-8-1EP_6x5mm_P1.27mm_EP3.4x4.3mm, symbol Memory_Flash:W25Q32JVZP
- removed U3: MIC5504-3.3YM5, Package_TO_SOT_SMD:SOT-23-5, symbol Regulator_Linear:MIC5504-3.3YM5
- added C40, C41, C43, C44, C46, C47, C48, C50, C52, C54, C55, C56: 100n, Capacitor_SMD:C_0603_1608Metric, symbol Device:C_Small
- added C42, C45, C49, C51, C53: 10n, Capacitor_SMD:C_0603_1608Metric, symbol Device:C_Small
- added D11, D12: LED, LED_SMD:LED_0805_2012Metric, symbol Device:LED
- added J4: Conn_01x22_Socket, Connector_PinSocket_2.54mm:PinSocket_1x22_P2.54mm_Horizontal, symbol Connector:Conn_01x22_Socket
- added R79, R80, R81, R82, R85, R86: 220R, Resistor_SMD:R_0603_1608Metric, symbol Device:R_Small_US
- added R83, R84: 100R, Resistor_SMD:R_0603_1608Metric, symbol Device:R_Small_US
- added SW0, SW1, SW2, SW3, SW4, SW5, SW6, SW7: ~, ProgrammaGull_Logic:SLW-121586-5A-D, symbol ProgrammaGull_Logic:SW_SPDT_W_CASE
- added U11: ADC084S051CIMM/NOPB, Package_SO:VSSOP-10_3x3mm_P0.5mm, symbol ProgrammaGull_Logic:ADC084S051CIMM/NOPB
- added U14: W25Q32JVSS, Package_SO:SOIC-8_5.23x5.23mm_P1.27mm, symbol Memory_Flash:W25Q32JVSS
- added U15: AMS1117-3.3, Package_TO_SOT_SMD:SOT-223-3_TabPin2, symbol Regulator_Linear:AMS1117-3.3
- added U2: SN74LVC1G126DCKR, ProgrammaGull_Logic:SC70, symbol ProgrammaGull_Logic:SN74LVC1G126DCKR
- added X1: SG-210STF, Oscillator:Oscillator_SMD_SeikoEpson_SG210-4Pin_2.5x2.0mm, symbol Oscillator:SG-210STF
- C1, C11, C13, C14, C16, C18, C19, C2, C20, C21, C22, C23, C24, C26, C28, C29, C3, C31, C32, C34, C36, C37, C38, C39, C4, C5, C6, C8, C9: footprint (none) -> Capacitor_SMD:C_0603_1608Metric
- C10, C12, C15, C17, C25, C27, C30, C33, C35, C7: footprint (none) -> Capacitor_SMD:C_0805_2012Metric
- D10: footprint (none) -> LED_SMD:LED_Cree-PLCC4_2x2mm_CW
- D2, D3, D4, D5, D6, D7, D8, D9: footprint (none) -> LED_SMD:LED_0805_2012Metric
- FB1, FB2: footprint (none) -> Inductor_SMD:L_0603_1608Metric
- P1: footprint (none) -> Connector_USB:USB_C_Receptacle_GCT_USB4105-xx-A_16P_TopMnt_Horizontal
- R1: value 27R -> 10k; footprint (none) -> Resistor_SMD:R_0603_1608Metric
- R10, R11, R12, R13, R14, R15, R16, R17, R18, R19, R20, R21, R22, R23, R24, R25, R26, R27, R28, R29, R3, R30, R31, R32, R33, R34, R36, R37, R38, R39, R4, R40, R41, R42, R43, R44, R45, R46, R47, R48, R49, R5, R50, R51, R52, R53, R54, R55, R56, R57, R58, R59, R6, R60, R61, R62, R63, R64, R65, R66, R67, R68, R69, R7, R70, R71, R72, R73, R74, R75, R76, R77, R78, R8, R9: footprint (none) -> Resistor_SMD:R_0603_1608Metric
- SW10, SW11, SW12, SW13, SW14, SW9: footprint (none) -> ProgrammaGull_Logic:Alps_SKQGAKE010
- SW15: footprint (none) -> Rotary_Encoder:RotaryEncoder_Bourns_Vertical_PEC12R-3xxxF-Nxxxx
- U10, U8: footprint (none) -> ProgrammaGull_Logic:MHDA3641SRBW
- U12, U13, U9: footprint (none) -> Package_SO:TSSOP-16_4.4x5mm_P0.65mm
Connections:
- net VBUS is gone; now on net +5V: C24.1, C25.1, C26.1, P1.A4 (VBUS), P1.A9 (VBUS), P1.B4 (VBUS), P1.B9 (VBUS), Q1.2 (E), Q2.2 (E), Q3.2 (E), Q4.2 (E), Q5.2 (E), Q6.2 (E), Q7.2 (E), Q8.2 (E), R67.2, R68.2, R69.2, R70.2, R71.2, R72.2, R73.2, R74.2
- net +1V2: now also C48.1, C49.1, C56.1
- net +1V8: now also C46.1, C47.1
- net +3V3: now also C2.1, C3.1, R1.2, U4.1 (VIN), U4.3 (EN), U5.1 (VIN), U5.3 (EN), C40.1, C41.1, C43.1, C44.1, C50.1, C51.1, C52.1, C53.1, C54.1, C55.1, J4.1 (Pin_1), J4.13 (Pin_13), J4.18 (Pin_18), J4.7 (Pin_7), SW0.1, SW1.1, SW2.1, SW3.1, SW4.1, SW5.1, SW6.1, SW7.1, U11.2 (VA), U14.8 (VCC), U15.2 (VO), U2.5 (VCC), X1.4 (Vcc)
- net +5V: now also U15.3 (VI); no longer C2.1, C3.1, U4.1 (VIN), U4.3 (EN), U5.1 (VIN), U5.3 (EN)
- net CLK_12M: now also U1.37 (IOT_45a_G1), U2.4 (Y)
- net FLASH_CS: now also U14.1 (~{CS})
- net FLASH_MISO: now also U14.2 (DO(IO1))
- net FLASH_MOSI: now also U14.5 (DI(IO0))
- net FLASH_SCK: now also U14.6 (CLK)
- net GND: now also C40.2, C41.2, C42.2, C43.2, C44.2, C45.2, C46.2, C47.2, C48.2, C49.2, C50.2, C51.2, C52.2, C53.2, C54.2, C55.2, C56.2, D11.1 (K), D12.1 (K), J4.15 (Pin_15), J4.17 (Pin_17), J4.20 (Pin_20), J4.22 (Pin_22), J4.6 (Pin_6), J4.8 (Pin_8), SW0.3, SW0.4 (CASE), SW1.3, SW1.4 (CASE), SW2.3, SW2.4 (CASE), SW3.3, SW3.4 (CASE), SW4.3, SW4.4 (CASE), SW5.3, SW5.4 (CASE), SW6.3, SW6.4 (CASE), SW7.3, SW7.4 (CASE), U11.3 (GND), U14.4 (GND), U15.1 (GND), U2.3 (GND), X1.2 (GND)
- net UI_7SEGSR_CLK: now also U1.13 (IOB_24a); no longer U1.11 (IOB_20a)
- net UI_7SEGSR_DIN: now also U1.11 (IOB_20a), U9.14 (SER); no longer U1.10 (IOB_18a), U12.14 (SER)
- net UI_7SEG_SER_CARRY: now also U12.14 (SER), U9.9 (QH'); no longer U12.9 (QH'), U9.14 (SER)
- net UI_DPAD_C: no longer U1.36 (IOT_48b)
- net UI_DPAD_L: now also U1.36 (IOT_48b); no longer U1.37 (IOT_45a_G1)
- net UI_LED_0: now also U13.7 (QH); no longer U13.15 (QA)
- net UI_LED_1: now also U13.6 (QG); no longer U13.1 (QB)
- net UI_LED_2: now also U13.5 (QF); no longer U13.2 (QC)
- net UI_LED_3: now also U13.4 (QE); no longer U13.3 (QD)
- net UI_LED_4: now also U13.3 (QD); no longer U13.4 (QE)
- net UI_LED_5: now also U13.2 (QC); no longer U13.5 (QF)
- net UI_LED_6: now also U13.1 (QB); no longer U13.6 (QG)
- net UI_LED_7: now also U13.15 (QA); no longer U13.7 (QH)
- net UI_LSB_CA0: now also U9.3 (QD); no longer U9.15 (QA)
- net UI_LSB_CA1: now also U9.2 (QC); no longer U9.1 (QB)
- net UI_LSB_CA2: now also U9.1 (QB); no longer U9.2 (QC)
- net UI_LSB_CA3: now also U9.15 (QA); no longer U9.3 (QD)
- net UI_MSB_CA0: now also U9.7 (QH); no longer U9.4 (QE)
- net UI_MSB_CA1: now also U9.6 (QG); no longer U9.5 (QF)
- net UI_MSB_CA2: now also U9.5 (QF); no longer U9.6 (QG)
- net UI_MSB_CA3: now also U9.4 (QE); no longer U9.7 (QH)
- net UI_ROTENC_A: no longer U1.19 (IOB_29b)
- net UI_ROTENC_B: no longer U1.18 (IOB_31b)
- net UI_ULEDSR_CLK: now also U1.21 (IOB_23b); no longer U1.20 (IOB_25b_G3)
- net UI_ULEDSR_DIN: now also U1.20 (IOB_25b_G3); no longer U1.21 (IOB_23b)
- net UP5K_UART_RX: now also U1.19 (IOB_29b)
- net UP5K_UART_TX: now also U1.18 (IOB_31b)
- net USB_D+: now also P1.A6 (D+)
- net USB_D-: now also P1.A7 (D-); no longer R1.2
- net ~{UI_7SEGSR_OE}: now also U1.10 (IOB_18a), U12.13 (~{OE}); no longer U1.13 (IOB_24a), U9.13 (~{OE})
- net at R10.1, R11.1: now also SW5.2
- net at R20.1, R21.1: now also SW0.2
- net at R14.1, R15.1: now also SW3.2
- net UI_GPIO0: now reaches U1.6 (IOB_13b)
- net UI_GPIO0: now also J4.14 (Pin_14), R83.2
- net UI_GPIO1: now reaches U1.9 (IOB_16a)
- net UI_GPIO1: now also J4.19 (Pin_19), R84.2
- net at R43.2: now also U12.7 (QH); no longer U12.15 (QA)
- net UI_PMOD0_1: now reaches U1.2 (IOB_6a)
- net UI_PMOD0_1: now also R81.2
- net UI_PMOD0_2: now reaches U1.3 (IOB_9b)
- net UI_PMOD0_2: now also R80.2
- net UI_PMOD0_3: now reaches U1.4 (IOB_8a)
- net UI_PMOD0_3: now also R79.2
- net ~{UI_ADC_CS}: now reaches U1.44 (IOB_3b_G6)
- net ~{UI_ADC_CS}: now also U11.1 (~{CS})
- net UI_ADC_SCK: now reaches U1.45 (IOB_5b)
- net UI_ADC_SCK: now also U11.10 (SCK)
- net UI_ADC_DO: now reaches U1.46 (IOB_0a)
- net UI_ADC_DO: now also U11.9 (DOUT)
- net UI_ADC_DI: now reaches U1.47 (IOB_2a)
- net UI_ADC_DI: now also U11.8 (DIN)
- net UI_PMOD0_0: now reaches U1.48 (IOB_4a)
- net UI_PMOD0_0: now also R82.2
- net at U12.1 (QB): now also R49.2; no longer R44.2
- net at R54.2: now also U9.13 (~{OE}); no longer U12.13 (~{OE})
- net at U12.2 (QC): now also R48.2; no longer R45.2
- net at U12.3 (QD): now also R47.2; no longer R46.2
- net at U12.4 (QE): now also R46.2; no longer R47.2
- net at U12.5 (QF): now also R45.2; no longer R48.2
- net at U12.6 (QG): now also R44.2; no longer R49.2
- net at R50.2: now also U12.15 (QA); no longer U12.7 (QH)
- net at R18.1, R19.1: now also SW1.2
- net at R6.1, R7.1: now also SW7.2
- net at U7.54 (BCBUS3): now also R86.2
- net at U7.55 (BCBUS4): now also R85.2
- net at R16.1, R17.1: now also SW2.2
- net at R40.1: now also U14.3 (IO2)
- net at R41.1: now also U14.7 (IO3)
- net at R1.1: now also U2.1 (OE); no longer P1.A7 (D-)
- net at R12.1, R13.1: now also SW4.2
- net at R8.1, R9.1: now also SW6.2
- new net: J4.10 (Pin_10), R81.1
- new net: J4.11 (Pin_11), R80.1
- new net: J4.12 (Pin_12), R79.1
- new net: C42.1, J4.16 (Pin_16), R83.1
- new net: C45.1, J4.21 (Pin_21), R84.1
- new net: J4.9 (Pin_9), R82.1
- new net: D12.2 (A), R86.1
- new net: U2.2 (A), X1.3 (OUT)
- new net: D11.2 (A), R85.1
- new net UI_ADC_SE_CHAN_0: J4.5 (Pin_5), U11.7 (IN1)
- new net UI_ADC_SE_CHAN_1: J4.4 (Pin_4), U11.6 (IN2)
- new net UI_ADC_SE_CHAN_2: J4.3 (Pin_3), U11.5 (IN3)
- new net UI_ADC_SE_CHAN_3: J4.2 (Pin_2), U11.4 (IN4)
- no-connect marks 24 -> 23
Other:
- note added: "6 pin PMOD interface :)"
- note added: "ADC"
- note added: "ADC - 4 input, 8 bit, 500ksps"
- note added: "Alt Part (Pin Compatible): ADC084S101CIMM/NOPB for 1MSPS"
- note added: "Analog Inputs (Unprotected!!)"
- note added: "Bougie: Panasonic EVP-ASAC1A"
- note added: "Can only drive 15pf, throw thru buffer :) -> SN74LVC1G126DCKR -> https://www.ti.com/lit/ds/symlink/sn74lvc1g126.pdf"
- note added: "EXT CLK"
- note added: "FTDI -> USB LED (TX)"
- note added: "For Case Option: Alps SKQGAKE010"
- note added: "GPIO + RCLP"
- note added: "GPIO 0, with RCLP Alias"
- note added: "GPIO 1, with RCLP Alias"
- note added: "Keep OE disabled such that CA transistors are disabled by default. Unused ports will be HI-Z inputs and as such will not drive the ~{OE} pin."
- note added: "OUT OF PINS NO USEY"
- note added: "PMOD"
- note added: "Removed MIC5504 3V3 for more current capacity"
- note added: "Single Ended, Single ADC w/ Mux input"
- note added: "USB -> FTDI LED (RX)"
- note added: "User Accessible Pins"
- note removed: "Keep OE disabled such that CA transistors are disabled by default."
- moved on the sheet: C36, R43, R44, R45, R46, R47, R48, R49, R50, R51, R53, R54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
