File: Boards/ProgrammaGull_Sandpiper/ProgrammaGull_Sandpiper_v_Alpha/ProgrammaGull_Sandpiper.kicad_sch (KiCad schematic)
At the start: 190 parts, among them J4 Conn_01x22_Socket, P1 USB_C_Plug_USB2.0, Q1 MMBT2907, Q2 MMBT2907, Q3 MMBT2907, Q4 MMBT2907, Q5 MMBT2907, Q6 MMBT2907, Q7 MMBT2907, Q8 MMBT2907, SW10 SW_Push, SW11 SW_Push, SW12 SW_Push, SW14 SW_Push, SW9 SW_Push, U1 ICE40UP5K-SG48ITR, U11 ADC084S051CIMM/NOPB, U12 74HC596, U13 74AHC595, U14 W25Q32JVSS, U15 AMS1117-3.3, U2 SN74LVC1G126DCKR, U3 74HC596, U4 MIC5504-1.2YM5, U5 MIC5504-2.5YM5, U6 93LCxxAxxOT, U7 FT2232HQ, X1 SG-210STF

Commit message: In progress conversion to maintaining 5V on seven segment
Parts:
- removed U3: 74HC596, Package_SO:TSSOP-16_4.4x5mm_P0.65mm, symbol 74xx:74HC596
- added Q10, Q11, Q12, Q13, Q14, Q15, Q16, Q9: MMBT3904, Package_TO_SOT_SMD:SOT-23, symbol Transistor_BJT:MMBT3904
- added R100, R101, R30, R31, R75, R76, R77, R78, R92, R93, R94, R95, R96, R97, R98, R99: 10k, Resistor_SMD:R_0603_1608Metric, symbol Device:R_Small_US
- added U9: 74AHC595, Package_SO:TSSOP-16_4.4x5mm_P0.65mm, symbol 74xx:74AHC595
Connections:
- net +3V3: now also U9.16 (VCC)
- net GND: now also R100.1, R101.1, R30.1, R31.1, R75.1, R76.1, R77.1, R78.1, R92.1, R93.1, R94.1, R95.1, R96.1, R97.1, R98.1, R99.1, U9.8 (GND)
- net UI_7SEGSR_CLK: now also U9.11 (SRCLK)
- net UI_7SEGSR_DIN: now also U9.14 (SER)
- net UI_7SEGSR_RCLK: now also U9.12 (RCLK)
- net UI_7SEG_SER_CARRY: now also U9.9 (QH')
- net UI_LSB_CA0: now also Q13.1 (B), R94.2; no longer Q5.1 (B), R71.1
- net UI_LSB_CA1: now also Q14.1 (B), R96.2; no longer Q6.1 (B), R72.1
- net UI_LSB_CA2: now also Q15.1 (B), R98.2; no longer Q7.1 (B), R73.1
- net UI_LSB_CA3: now also Q16.1 (B), R100.2; no longer Q8.1 (B), R74.1
- net UI_MSB_CA0: now also Q9.1 (B), R30.2; no longer Q1.1 (B), R67.1
- net UI_MSB_CA1: now also Q10.1 (B), R75.2; no longer Q2.1 (B), R68.1
- net UI_MSB_CA2: now also Q11.1 (B), R77.2; no longer Q3.1 (B), R70.1
- net UI_MSB_CA3: now also Q12.1 (B), R92.2; no longer Q4.1 (B), R69.1
- net ~{UI_7SEGSR_OE}: now also U9.13 (~{OE})
- net at R35.2: now also U9.7 (QH)
- net at R54.2: now also U9.2 (QC)
- net at R89.2: now also U9.5 (QF)
- net at C36.1, R51.1: now also U9.10 (~{SRCLR})
- net at R90.2: now also U9.15 (QA)
- net at R87.2: now also U9.6 (QG)
- net at R2.2: now also U9.3 (QD)
- net at R88.2: now also U9.1 (QB)
- net at R91.2: now also U9.4 (QE)
- new net: Q15.2 (E), R99.2
- new net: Q16.2 (E), R101.2
- new net: Q13.2 (E), R95.2
- new net: Q14.2 (E), R97.2
- new net: Q11.2 (E), R78.2
- new net: Q10.2 (E), R76.2
- new net: Q12.2 (E), R93.2
- new net: Q9.2 (E), R31.2
- new net CA0_LSB_BASE: Q13.3 (C), Q5.1 (B), R71.1
- new net CA0_MSB_BASE: Q1.1 (B), Q9.3 (C), R67.1
- new net CA1_LSB_BASE: Q14.3 (C), Q6.1 (B), R72.1
- new net CA1_MSB_BASE: Q10.3 (C), Q2.1 (B), R68.1
- new net CA2_LSB_BASE: Q15.3 (C), Q7.1 (B), R73.1
- new net CA2_MSB_BASE: Q11.3 (C), Q3.1 (B), R70.1
- new net CA3_LSB_BASE: Q16.3 (C), Q8.1 (B), R74.1
- new net CA3_MSB_BASE: Q12.3 (C), Q4.1 (B), R69.1
Other:
- note added: "Note: THIS IS PUSH-PULL"
- moved on the sheet: C36, C37, C40, C41, C42, C43, C44, C45, C50, C51, C52, C53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
