File: Boards/ProgrammaGull_Sandpiper/PGL_Sandpiper_v_1/ProgrammaGull_Sandpiper.kicad_pcb (KiCad board)
At the start: 4 copper layers, 100 x 75 mm, 214 parts, among them J1 Conn_02x14_Odd_Even, P1 USB_C_Plug_USB2.0, Q1 S9012 2T1, Q2 S9012 2T1, Q3 S9012 2T1, Q4 S9012 2T1, Q5 S9012 2T1, Q6 S9012 2T1, Q7 S9012 2T1, Q8 S9012 2T1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

Commit message: Final revision Sandpiper V1, sent for fab
Parts:
- moved C42 5.33 mm to (108.5, 39.1)
- moved C44 5.33 mm to (109.2, 56.9)
- moved C45 5.33 mm to (108.5, 42.2)
- moved R93 5.33 mm to (109.0, 48.3)
- moved R94 5.33 mm to (109.0, 50.8)
- moved C41 5.33 mm to (108.4, 32.0)
- moved C43 5.33 mm to (108.5, 35.6)
- moved J1 5.33 mm to (112.3, 66.0)
- moved R83 5.33 mm to (108.5, 40.6)
- moved R84 5.33 mm to (108.5, 43.7)
- moved R92 5.33 mm to (109.0, 45.7)
- moved R95 5.33 mm to (109.0, 53.3)
- moved R96 5.33 mm to (109.0, 54.6)
- moved R97 5.33 mm to (109.0, 52.1)
- moved R98 5.33 mm to (109.0, 49.5)
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Routing:
- net /UI_GPIO0: track 50.3 -> 55.7 mm
- net +5V: track 198.0 -> 202.4 mm
- net /UI_GPIO1: track 46.8 -> 50.9 mm
- net /UI_ADC_SCK: track 27.1 -> 30.2 mm
- net /UI_PMOD0_2: track 35.0 -> 37.2 mm
- net /UI_PMOD0_3: track 32.2 -> 34.4 mm
- net /UI_PMOD0_1: track 36.3 -> 38.5 mm
- net /UI_PMOD0_0: track 37.4 -> 39.7 mm
- net /UI_ADC_DO: track 37.4 -> 39.6 mm
- net /~{UI_ADC_CS}: track 29.6 -> 27.5 mm
- net +3V3: track 149.3 -> 148.3 mm
- net /UI_ADC_DI: track 37.5 -> 38.1 mm
- net GND: track 92.9 -> 92.4 mm
