File: Boards/ProgrammaGull_Sandpiper/PGL_Sandpiper_v_1/ProgrammaGull_Sandpiper.kicad_sch (KiCad schematic)
At the start: 213 parts, among them J1 Conn_02x14_Odd_Even, P1 USB_C_Plug_USB2.0, Q1 S9012 2T1, Q2 S9012 2T1, Q3 S9012 2T1, Q4 S9012 2T1, Q5 S9012 2T1, Q6 S9012 2T1, Q7 S9012 2T1, Q8 S9012 2T1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

Commit message: Final revision Sandpiper V1, sent for fab
Connections:
- net GND: now also J1.20 (Pin_20)
Changed lines of the file:
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@@
     (stroke (width 0) (type default))
   )
-  (wire (pts (xy 647.7 265.43) (xy 648.97 265.43))
+  (wire (pts (xy 645.16 265.43) (xy 648.97 265.43))
     (stroke (width 0) (type default))
   )
