File: Boards/PGL_FTDI_Programmer/PGL_FTDI_Prog/PGL_FTDI_Prog.kicad_pcb (KiCad board)
At the start: 4 copper layers, 48 x 22 mm, 47 parts, among them J1 Conn_01x03_Pin, J3 Conn_01x04, P1 USB_C_Plug_USB2.0, U1 XC6206PxxxMR, U4 93LCxxAxxOT, U5 FT2232HQ, U6 PG Logic Full Size Programmin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, U7 PG_Logic_10_Pin_Tag_Connect_P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, Y1 12.000 MHz, C9002

Commit message: PGL Programmer Test Run Finished
Parts:
- removed U6: PG Logic Full Size Programming Interface, Connector_PinHeader_2.54mm:PinHeader_1x08_P2.54mm_Horizontal
- added G***: LOGO, LOGO, B.Cu at (82.6, 58.4)
- moved J1 0.64 mm to (100.2, 50.9)
Routing:
- net Net-(J1-Pin_2): track 11.0 -> 17.1 mm
- net +5V: track 83.1 -> 82.5 mm
Other:
- board size 48 x 22 mm -> 42 x 22 mm
- board text added: "3V"
- board text added: "FT2232HQ"
- board text removed: "3V3"
