File: Boards/PGL_E6/ProgrammaGull_E6/ProgrammaGull_E6.kicad_pcb (KiCad board)
At the start: 4 copper layers, 25.4 x 25.4 mm, 32 parts, among them U1 AMS1117-3.3, U2 MIC5504-2.5YM5, U3 MIC5504-1.2YM5, U4 W25Q32JVSS, U5 ICE40UP5K-SG48ITR, U6 PG_Logic_10_Pin_Tag_Connect, U7 W25Q16JVUXIQ_TR, U8 PGL_E6

Commit message: E6 layout redo
Parts:
- removed U6: PG_Logic_10_Pin_Tag_Connect, Connector:Tag-Connect_TC2050-IDC-NL_2x05_P1.27mm_Vertical
- removed U7: W25Q16JVUXIQ_TR, ICDB_Curly:IC_W25Q16JVUXIQ_TR
- removed U8: PGL_E6, ProgrammaGull_Logic:PGL_E6
- added JP1: SolderJumper_3_Open, Jumper:SolderJumper-3_P2.0mm_Open_TrianglePad1.0x1.5mm, F.Cu at (152.2, 85.9)
- added U9: AP7375-33SA-7, Package_TO_SOT_SMD:SOT-23-3, F.Cu at (157.0, 84.9)
- U1: value AMS1117-3.3 -> PGL_E6; footprint Package_TO_SOT_SMD:SOT-223-3_TabPin2 -> ProgrammaGull_Logic:PGL_E6
- moved D2 48.6 mm to (153.5, 83.5)
- moved U3 48.5 mm to (159.5, 89.0)
- moved U2 44.8 mm to (154.5, 89.0), turned to 180 degrees
- moved U5 43.6 mm to (157.0, 90.0), turned to 135 degrees
- moved U1 42.6 mm to (157.0, 90.0)
- moved C14 40.0 mm to (176.6, 91.9)
- moved C17 40.0 mm to (176.6, 99.4)
- moved C19 40.0 mm to (176.6, 104.5)
- moved C22 40.0 mm to (180.6, 91.9)
- moved C3 40.0 mm to (172.5, 96.9)
- moved R2 40.0 mm to (180.6, 96.9)
- moved R7 40.0 mm to (180.6, 104.5)
- moved C13 40.0 mm to (172.5, 109.5)
- moved C15 40.0 mm to (176.6, 94.4)
- moved C18 40.0 mm to (176.6, 101.9)
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Connections:
- net /BANK_0_VCC renamed Net-(JP1-C)
- U5 pad 10: unconnected-(U5B-IOB_18a-Pad10) -> /BANK_1_18A
- U5 pad 11: unconnected-(U5B-IOB_20a-Pad11) -> /BANK_1_20A
- U5 pad 12: unconnected-(U5B-IOB_22a-Pad12) -> /BANK_1_22A
- U5 pad 13: unconnected-(U5B-IOB_24a-Pad13) -> /BANK_1_24A
- U5 pad 18: /UP5K_UART_TX -> /BANK_1_31B
- U5 pad 19: /UP5K_UART_RX -> /BANK_1_29B
- U5 pad 20: unconnected-(U5B-IOB_25b_G3-Pad20) -> /BANK_1_25B_G3
- U5 pad 21: unconnected-(U5B-IOB_23b-Pad21) -> /BANK_1_23B
- U5 pad 23: unconnected-(U5A-IOT_37a-Pad23) -> /BANK_0_37A
- U5 pad 25: unconnected-(U5A-IOT_36b-Pad25) -> /BANK_0_36B
- U5 pad 26: unconnected-(U5A-IOT_39a-Pad26) -> /BANK_0_39A
- U5 pad 27: unconnected-(U5A-IOT_38b-Pad27) -> /BANK_0_38B
- U5 pad 28: unconnected-(U5A-IOT_41a-Pad28) -> /BANK_0_41A
- U5 pad 39: unconnected-(U5A-RGB0-Pad39) -> /RGB0
- U5 pad 40: unconnected-(U5A-RGB1-Pad40) -> /RGB1
- U5 pad 41: unconnected-(U5A-RGB2-Pad41) -> /RGB2
- U5 pad 6: unconnected-(U5B-IOB_13b-Pad6) -> /BANK_1_13B
- U5 pad 9: unconnected-(U5B-IOB_16a-Pad9) -> /BANK_1_16A
Routing:
- net +3V3: track 0.00 -> 42.0 mm, vias 6 -> 2
- net +2V5: track 0.00 -> 15.2 mm, vias 0 -> 1
- net /BANK_1_31B: track 0.00 -> 13.6 mm
- net GND: track 2.44 -> 14.9 mm, vias 7 -> 5
- net /BANK_1_16A: track 0.00 -> 11.6 mm
- net /BANK_1_29B: track 0.00 -> 11.6 mm
- net /BANK_1_25B_G3: track 0.00 -> 10.3 mm
- net /BANK_0_46B: track 9.92 -> 0.00 mm, vias 1 -> 0
- net /BANK_1_20A: track 0.00 -> 9.69 mm
- net /BANK_1_13B: track 0.00 -> 9.57 mm
- net /BANK_1_23B: track 0.00 -> 9.05 mm
- net /BANK_1_24A: track 0.00 -> 8.84 mm
- net /BANK_0_37A: track 0.00 -> 8.83 mm
- net /BANK_0_36B: track 0.00 -> 8.40 mm
- net +5V: track 15.1 -> 6.99 mm
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- removed copper zone on F.Cu, net GND
