File: Boards/PGL_E6/ProgrammaGull_E6/ProgrammaGull_E6.kicad_sch (KiCad schematic)
At the start: 32 parts, among them U1 AMS1117-3.3, U2 MIC5504-2.5YM5, U3 MIC5504-1.2YM5, U4 W25Q32JVSS, U5 ICE40UP5K-SG48ITR, U6 PG_Logic_10_Pin_Tag_Connect, U7 W25Q16JVUXIQ_TR, U8 PGL_E6

Commit message: E6 layout redo
Parts:
- removed U1: AMS1117-3.3, Package_TO_SOT_SMD:SOT-223-3_TabPin2, symbol Regulator_Linear:AMS1117-3.3
- removed U6: PG_Logic_10_Pin_Tag_Connect, Connector:Tag-Connect_TC2050-IDC-NL_2x05_P1.27mm_Vertical, symbol ProgrammaGull_Logic:PG_Logic_10_Pin_Tag_Connect
- removed U7: W25Q16JVUXIQ_TR, ICDB_Curly:IC_W25Q16JVUXIQ_TR, symbol ICDB_Curly:W25Q16JVUXIQ_TR
- removed U8: PGL_E6, ProgrammaGull_Logic:PGL_E6, symbol ProgrammaGull_Logic:PGL_E6
- added JP1: SolderJumper_3_Open, Jumper:SolderJumper-3_P2.0mm_Open_TrianglePad1.0x1.5mm, symbol Jumper:SolderJumper_3_Open
- added U1: PGL_E6, ProgrammaGull_Logic:PGL_E6, symbol ProgrammaGull_Logic:PGL_E6
- added U9: AP7375-33SA-7, Package_TO_SOT_SMD:SOT-23-3, symbol ICDB_Waffle:AP7375-33SA-7
Connections:
- net +2V5: now also JP1.1 (A), U1.3C
- net +3V3: now also JP1.3 (B), U1.3I, U1.3J, U9.2 (VOUT)
- net +5V: now also U1.6A, U1.6B, U9.1 (VIN)
- net FLASH_CS: now also U1.4J
- net FLASH_MISO: now also U1.4I
- net FLASH_MOSI: now also U1.5J
- net FLASH_SCK: now also U1.5I
- net GND: now also U1.2H, U1.2I, U1.2J, U1.5A, U1.5B, U9.3 (GND)
- net UP5K_CDONE: now also U1.6J
- net ~{UP5K_CRESET}: now also U1.6I
- net BANK_1_18A: now reaches U5.10 (IOB_18a)
- net BANK_1_18A: now also U1.8I
- net BANK_1_20A: now reaches U5.11 (IOB_20a)
- net BANK_1_20A: now also U1.8J
- net BANK_1_22A: now reaches U5.12 (IOB_22a)
- net BANK_1_22A: now also U1.7I
- net BANK_1_24A: now reaches U5.13 (IOB_24a)
- net BANK_1_24A: now also U1.7J
- net BANK_1_25B_G3: now reaches U5.20 (IOB_25b_G3)
- net BANK_1_25B_G3: now also U1.1H
- net BANK_1_23B: now reaches U5.21 (IOB_23b)
- net BANK_1_23B: now also U1.1G
- net BANK_1_13B: now reaches U5.6 (IOB_13b)
- net BANK_1_13B: now also U1.9I
- net BANK_1_16A: now reaches U5.9 (IOB_16a)
- net BANK_1_16A: now also U1.9J
- net BANK_0_37A: now reaches U5.23 (IOT_37a)
- net BANK_0_37A: now also U1.1F
- net BANK_0_36B: now reaches U5.25 (IOT_36b)
- net BANK_0_36B: now also U1.1E
- net BANK_0_39A: now reaches U5.26 (IOT_39a)
- net BANK_0_38B: now reaches U5.27 (IOT_38b)
- net BANK_0_41A: now reaches U5.28 (IOT_41a)
- net RGB0: now reaches U5.39 (RGB0)
- net RGB1: now reaches U5.40 (RGB1)
- net RGB2: now reaches U5.41 (RGB2)
- net BANK_0_VCC: no longer names the net of C18.1, C20.1, U5.33 (VCCIO_0)
- net BANK_0_VCC: now also JP1.2 (C)
- net UP5K_UART_RX renamed BANK_1_29B
- net BANK_1_29B: now also U1.1I
- net UP5K_UART_TX renamed BANK_1_31B
- net BANK_1_31B: now also U1.1J
